File: test/footprints/rest___pcbs_pcb.kicad_pcb (KiCad board)
At the start: 2 copper layers, 19.6 x 14.2 mm, 12 parts, among them J1 Jumper

Commit message: ✅ Fix tests
Parts:
- J1: footprint PCM12SMTR -> Jumper:SolderJumper-2_P1.3mm_Open_TrianglePad1.0x1.5mm
