File: test/pcbs/mock_footprints___pcbs_main.kicad_pcb (KiCad board)
At the start: 2 copper layers, 39 x 19 mm, 11 parts

Commit message: ✅ Fix tests
Parts:
- removed the ? at (0.00, 0.00) (x7)
- added ? (x2): , anchor_test, F.Cu at (0.00, 0.00)
- added ? (x2): , arrobj_test, F.Cu at (0.00, 0.00)
Changed lines of the file:
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@@
 (kicad_pcb (version 20211014) (generator pcbnew)
-  (general
-    (thickness 1.6)
-  )
   (paper "A3")
   (title_block
@@
     (rev "v1.0.0")
     (company "Unknown")
+  )
+  (general
+    (thickness 1.6)
   )
   (layers
@@
     (visible_elements FFFFFF7F)
     (pcbplotparams
-      (layerselection 0x00010fc_ffffffff)
-      (disableapertmacros false)
+      (layerselection 0x010fc_ffffffff)
       (usegerberextensions false)
       (usegerberattributes true)
       (usegerberadvancedattributes true)
       (creategerberjobfile true)
-      (svguseinch false)
-      (svgprecision 6)
       (excludeedgelayer true)
+      (linewidth 0.100000)
       (plotframeref false)
       (viasonmask false)
@@
       (hpglpenspeed 20)
       (hpglpendiameter 15.000000)
-      (dxfpolygonmode true)
-      (dxfimperialunits true)
-      (dxfusepcbnewfont true)
       (psnegative false)
       (psa4output false)
@@
       (plotvalue true)
       (plotinvisibletext false)
-      (sketchpadsonfab false)
+      (padsonsilk false)
       (subtractmaskfromsilk false)
       (outputformat 1)
@@
       (drillshape 1)
       (scaleselection 1)
-      (outputdirectory "")
-    )
+      (outputdirectory ""))
   )
             (net 0 "")
@@
 (add_net "T4_2")
 (add_net "T4_3")
-  )
-  (net_class Power "This is the power net class."
-    (clearance 0.2)
-    (trace_width 0.5)
-    (via_dia 0.8)
-    (via_drill 0.4)
-    (uvia_dia 0.3)
-    (uvia_drill 0.1)
   )
   (net_class Power "This is the power net class."
@@
                 )
                 (module anchor_test (layer F.Cu)
-                    (at 0 0 0)
-                    (fp_line (start 0 0) (end 0 0) (layer Dwgs.User) (width 0.05))
-                )
-                (module arrobj_test (layer F.Cu)
-                    (at 0 0 0)
-                    (fp_line (start 5 5) (end 6 6) (layer Dwgs.User) (width 0.05))
-(fp_line (start 5 5) (end 7 7) (layer Dwgs.User) (width 0.05))
-                )
-                (module arrobj_test (layer F.Cu)
-                    (at 0 0 0)
-                    (fp_line (start 5 5) (end 6 6) (layer Dwgs.User) (width 0.05))
-(fp_line (start 5 5) (end 7 5) (layer Dwgs.User) (width 0.05))
-                )
-                (module anchor_test (layer F.Cu)

Commit message: Update to Kicad 7 format
Parts:
- removed the ? at (0.00, 0.00) (x4)
- added ? (x2): , anchor_test, F.Cu at (0.00, 0.00)
- added ? (x2): , arrobj_test, F.Cu at (0.00, 0.00)
Changed lines of the file:
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@@
-(kicad_pcb (version 20211014) (generator pcbnew)
+(kicad_pcb (version 20221018) (generator pcbnew)
+  (general
+    (thickness 1.6)
+  )
   (paper "A3")
   (title_block
@@
     (rev "v1.0.0")
     (company "Unknown")
-  )
-  (general
-    (thickness 1.6)
   )
   (layers
@@
     (pcbplotparams
       (layerselection 0x010fc_ffffffff)
+      (disableapertmacros false)
       (usegerberextensions false)
       (usegerberattributes true)
       (usegerberadvancedattributes true)
       (creategerberjobfile true)
+      (svguseinch false)
+      (svgprecision 6)
       (excludeedgelayer true)
-      (linewidth 0.100000)
       (plotframeref false)
       (viasonmask false)
@@
       (hpglpenspeed 20)
       (hpglpendiameter 15.000000)
+      (dxfpolygonmode true)
+      (dxfimperialunits true)
+      (dxfusepcbnewfont true)
       (psnegative false)
       (psa4output false)
@@
       (plotvalue true)
       (plotinvisibletext false)
-      (padsonsilk false)
+      (sketchpadsonfab false)
       (subtractmaskfromsilk false)
       (outputformat 1)

Commit message: Update format to Kicad 7 - continued
Parts:
- removed the ? at (0.00, 0.00) (x4)
- added ? (x2): , anchor_test, F.Cu at (0.00, 0.00)
- added ? (x2): , arrobj_test, F.Cu at (0.00, 0.00)
Changed lines of the file:
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@@
     (visible_elements FFFFFF7F)
     (pcbplotparams
-      (layerselection 0x010fc_ffffffff)
+      (layerselection 0x00010fc_ffffffff)
+      (plot_on_all_layers_selection 0x0000000_00000000)
       (disableapertmacros false)
       (usegerberextensions false)
@@
       (usegerberadvancedattributes true)
       (creategerberjobfile true)
-      (svguseinch false)
+      (dashed_line_dash_ratio 12.000000)
+      (dashed_line_gap_ratio 3.000000)
       (svgprecision 6)
-      (excludeedgelayer true)
       (plotframeref false)
       (viasonmask false)
@@
       (drillshape 1)
       (scaleselection 1)
-      (outputdirectory ""))
+      (outputdirectory "")
+    )
   )
             (net 0 "")
